Commit message: Correct configs and launch files for running gripper and screwdriver

File: epos_hardware/launch/gripper.urdf (robot description, URDF)
Before this commit: robot example, 2 links, 1 joints
Links:
- removed link link1
- removed link link2
- added link gripper_base_link, mass 1
- added link gripper_ee_link, mass 1
Joints:
- removed joint test_joint
- added joint gripper_joint: type revolute, parent gripper_base_link, child gripper_ee_link

File: epos_hardware/launch/screwdriver.urdf (robot description, URDF)
Before this commit: robot example, 2 links, 1 joints
Links:
- removed link link1
- removed link link2
- added link screwdriver_base_link, mass 1
- added link screwdriver_ee_link, mass 1
Joints:
- removed joint test_joint
- added joint screwdriver_joint: type revolute, parent screwdriver_base_link, child screwdriver_ee_link
